File: hardware/mh-custom-v2/mh-custom-v2.kicad_pcb (KiCad board)
At the start: 2 copper layers, 95.7 x 99.3 mm, 117 parts, among them J1 Conn_01x03_Male, J10 Screw_Terminal_01x02, J11 Screw_Terminal_01x02, J12 Screw_Terminal_01x02, J3 Conn_02x19_Top_Bottom, J4 Conn_02x19_Top_Bottom, J5 Screw_Terminal_01x02, J6 Screw_Terminal_01x02, J7 Screw_Terminal_01x02, J8 Screw_Terminal_01x02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

Commit message: just ordered from JLCPCB
Other:
- board text added: "'H'=H/L1 && 'N'=N/L2"
- board text added: "3 stages or relays WiFi microcontroller E-Stop Integration Current Sensor"
- board text added: "Best when used with ESPHome & Home Assistant"
- board text added: "Hot/L1"
- board text added: "Out to Stage 3 Contactor"
- board text added: "Set DIP switches for board-config"
- board text added: "Stage 1"
- board text added: "Stage 2"
- board text removed: "3 stages or relays WiFi microcontroller E-Stop integration Current Sensor"
- board text removed: "H/L1"
- board text removed: "Set DIP switches for board-config in ESPHome GUI"
