File: hardware/mh-custom-v2/stage1relays.kicad_sch (KiCad schematic)
At the start: 14 parts, among them T3 AO3400A, T4 AO3400A

Commit message: approaching ordering from JLCPCB
Parts:
- 5vRelay1-1, 5vRelay1-2: JLCPCB Part # (none) -> C35449
- D3, D4: JLCPCB Part # (none) -> C24784
- R26, R27, R29: JLCPCB Part # (none) -> C21190
- R28, R30: JLCPCB Part # (none) -> C25804
- T3, T4: JLCPCB Part # (none) -> C427382
Changed lines of the file:
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@@
   (symbol (lib_id "Device:R_US") (at 118.11 106.68 0) (unit 1)
     (in_bom yes) (on_board yes)
-    (property "Reference" "R28" (id 0) (at 114.3 107.95 0)
+    (property "Reference" "R28" (id 0) (at 113.03 107.95 0)
       (effects (font (size 1.27 1.27)) (justify left))
     )
@@
     )
     (property "Datasheet" "~" (id 3) (at 118.11 106.68 0)
+      (effects (font (size 1.27 1.27)) hide)
+    )
+    (property "JLCPCB Part #" "C25804" (id 4) (at 118.11 106.68 0)
       (effects (font (size 1.27 1.27)) hide)
     )
@@
       (effects (font (size 1.27 1.27)) hide)
     )
+    (property "JLCPCB Part #" "C35449" (id 4) (at 132.08 85.09 0)
+      (effects (font (size 1.27 1.27)) hide)
+    )
     (pin "1")
     (pin "2")
@@
       (effects (font (size 1.27 1.27)) hide)
     )
+    (property "JLCPCB Part #" "C21190" (id 4) (at 54.61 80.01 90)
+      (effects (font (size 1.27 1.27)) hide)
+    )
     (pin "1")
     (pin "2")
@@
       (effects (font (size 1.27 1.27)) hide)
     )
+    (property "JLCPCB Part #" "C21190" (id 4) (at 114.3 102.87 90)
+      (effects (font (size 1.27 1.27)) hide)
+    )
     (pin "1")
     (pin "2")
@@
       (effects (font (size 1.27 1.27)) hide)
     )
+    (property "JLCPCB Part #" "C24784" (id 4) (at 118.11 85.09 90)
+      (effects (font (size 1.27 1.27)) hide)
+    )
     (pin "1")
     (pin "2")
@@
     (property "Datasheet" "http://www.aosmd.com/pdfs/datasheet/AO3400A.pdf" (id 3) (at 124.46 102.87 0)
       (effects (font (size 1.27 1.27)) (justify left) hide)
+    )
+    (property "JLCPCB Part #" "C427382" (id 4) (at 124.46 102.87 0)
+      (effects (font (size 1.27 1.27)) hide)
     )
     (pin "1")
@@
       (effects (font (size 1.27 1.27)) hide)
     )
+    (property "JLCPCB Part #" "C21190" (id 4) (at 196.85 102.87 90)
+      (effects (font (size 1.27 1.27)) hide)
+    )
     (pin "1")
     (pin "2")
@@
     )
     (property "Datasheet" "http://www.vishay.com/docs/88946/b120.pdf" (id 3) (at 200.66 86.36 0)
+      (effects (font (size 1.27 1.27)) hide)
+    )
+    (property "JLCPCB Part #" "C24784" (id 4) (at 200.66 86.36 90)
       (effects (font (size 1.27 1.27)) hide)
     )
@@
     )
     (property "Datasheet" "http://www.sanyourelay.ca/public/products/pdf/SRD.pdf" (id 3) (at 214.63 86.36 0)
+      (effects (font (size 1.27 1.27)) hide)
+    )
+    (property "JLCPCB Part #" "C35449" (id 4) (at 214.63 86.36 0)
       (effects (font (size 1.27 1.27)) hide)
     )
@@
       (effects (font (size 1.27 1.27)) hide)
     )
+    (property "JLCPCB Part #" "C25804" (id 4) (at 200.66 106.68 0)
+      (effects (font (size 1.27 1.27)) hide)
+    )
     (pin "1")
     (pin "2")
@@
       (effects (font (size 1.27 1.27)) (justify left) hide)
     )
-    (pin "1")
+    (property "JLCPCB Part #" "C427382" (id 4) (at 207.01 102.87 0)
+      (effects (font (size 1.27 1.27)) hide)
+    )
+    (pin "1")

Commit message: prepping for JLCPCB order - all parts listed with numbers, BOM generated
Parts:
- Bypass-1: JLCPCB Part # (none) -> C131337
- D2: JLCPCB Part # (none) -> C2286
Changed lines of the file:
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@@
+      (effects (font (size 1.27 1.27)) hide)
+    )
+    (property "JLCPCB Part #" "C2286" (id 4) (at 54.61 86.36 90)
       (effects (font (size 1.27 1.27)) hide)
     )
@@
       (effects (font (size 1.27 1.27)) hide)
     )
+    (property "JLCPCB Part #" "C131337" (id 4) (at 152.4 101.6 0)
+      (effects (font (size 1.27 1.27)) hide)
+    )
