File: hardware/mh-custom-v2/_autosave-stage1relays.kicad_sch (KiCad schematic)
At the start: 14 parts, among them T3 AO3400A, T4 AO3400A

Commit message: finalizing details of ordering from JLCPCB
Parts:
- 5vRelay-1: footprint Relay_THT:Relay_SPDT_Omron-G5LE-1 -> Relay_THT:Relay_SPDT_SANYOU_SRD_Series_Form_C
Changed lines of the file:
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@@
       (effects (font (size 1.27 1.27)) (justify left))
     )
-    (property "Footprint" "Relay_THT:Relay_SPDT_Omron-G5LE-1" (id 2) (at 143.51 86.36 0)
+    (property "Footprint" "Relay_THT:Relay_SPDT_SANYOU_SRD_Series_Form_C" (id 2) (at 143.51 86.36 0)
       (effects (font (size 1.27 1.27)) (justify left) hide)
     )
@@
       (effects (font (size 1.27 1.27)) (justify left) hide)
     )
-    (property "Datasheet" "http://www.sanyourelay.ca/public/products/pdf/SRD.pdf" (id 3) (at 214.63 86.36 0)
-      (effects (font (size 1.27 1.27)) hide)
-    )
+    (property "Datasheet" "https://datasheet.lcsc.com/lcsc/2109061830_HF-Xiamen-Hongfa-Electroacoustic-JQC-3FF-005-1ZS-551_C9221.pdf" (id 3) (at 214.63 86.36 0)
+      (effects (font (size 1.27 1.27)) hide)
+    )
