File: hardware/mh-custom-v2/ade7953.kicad_sch (KiCad schematic)
At the start: 58 parts, among them U2 ADE7953xCP, Y1 3.58MHz

Commit message: added linear regulator for 3.3V peripherals and ADE7953 reset jumper
Parts:
- added JP13: software-reset, Jumper:SolderJumper-2_P1.3mm_Open_RoundedPad1.0x1.5mm, symbol Jumper:SolderJumper_2_Open
Connections:
- net ade7953-reset: now also JP13.1 (A); no longer C15.2, R22.1, U2.2 (~{RESET})
- new net: C15.2, JP13.2 (B), R22.1, U2.2 (~{RESET})
Changed lines of the file:
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@@
+    (stroke (width 0) (type default) (color 0 0 0 0))
+  )
+  (wire (pts (xy 119.38 72.39) (xy 120.65 72.39))
+    (stroke (width 0) (type default) (color 0 0 0 0))
+  )
+  (wire (pts (xy 163.83 106.68) (xy 180.34 106.68))
+    (stroke (width 0) (type default) (color 0 0 0 0))
+  )
+  (wire (pts (xy 179.07 118.11) (xy 181.61 118.11))
+    (stroke (width 0) (type default) (color 0 0 0 0))
+  )
+  (wire (pts (xy 66.04 54.61) (xy 64.77 54.61))
+    (stroke (width 0) (type default) (color 0 0 0 0))
+  )
+  (wire (pts (xy 77.47 181.61) (xy 77.47 185.42))
     (stroke (width 0) (type default) (color 0 0 0 0))
   )
   (wire (pts (xy 128.27 72.39) (xy 132.08 72.39))
-    (stroke (width 0) (type default) (color 0 0 0 0))
-  )
-  (wire (pts (xy 163.83 106.68) (xy 180.34 106.68))
-    (stroke (width 0) (type default) (color 0 0 0 0))
-  )
-  (wire (pts (xy 179.07 118.11) (xy 181.61 118.11))
-    (stroke (width 0) (type default) (color 0 0 0 0))
-  )
-  (wire (pts (xy 66.04 54.61) (xy 64.77 54.61))
-    (stroke (width 0) (type default) (color 0 0 0 0))
-  )
-  (wire (pts (xy 77.47 181.61) (xy 77.47 185.42))
     (stroke (width 0) (type default) (color 0 0 0 0))
   )
@@
     )
   )
-  (global_label "ade7953-reset" (shape input) (at 128.27 72.39 180) (fields_autoplaced)
+  (global_label "ade7953-reset" (shape input) (at 119.38 72.39 180) (fields_autoplaced)
     (effects (font (size 1 1)) (justify right))
-    (property "Intersheet References" "${INTERSHEET_REFS}" (id 0) (at 114.9414 72.3275 0)
+    (property "Intersheet References" "${INTERSHEET_REFS}" (id 0) (at 106.0514 72.3275 0)
       (effects (font (size 1 1)) (justify right) hide)
     )
@@
     (pin "1")
   )
+  (symbol (lib_id "Jumper:SolderJumper_2_Open") (at 124.46 72.39 0) (unit 1)
+    (in_bom yes) (on_board yes)
+    (property "Reference" "JP13" (id 0) (at 124.46 74.93 0))
+    (property "Value" "software-reset" (id 1) (at 124.46 77.47 0))
+    (property "Footprint" "Jumper:SolderJumper-2_P1.3mm_Open_RoundedPad1.0x1.5mm" (id 2) (at 124.46 72.39 0)
+      (effects (font (size 1.27 1.27)) hide)
+    )
+    (property "Datasheet" "~" (id 3) (at 124.46 72.39 0)
+      (effects (font (size 1.27 1.27)) hide)
+    )
+    (pin "1")
+    (pin "2")
+  )
   (symbol (lib_id "Device:R_Small_US") (at 48.26 88.9 270) (unit 1)
