File: hardware/mh-custom-v2/breakoutbaords.kicad_sch (KiCad schematic)
At the start: 8 parts, among them J3 Conn_02x19_Top_Bottom, J4 Conn_02x19_Top_Bottom, U3 AMS1117-3.3

Commit message: applied workaround for 3.3v and 3v3 known bug: https://gitlab.com/kicad/libraries/kicad-symbols/-/issues/3153
Connections:
- net +3V3 renamed +3.3VA
Changed lines of the file:
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@@
     (stroke (width 0) (type default) (color 0 0 0 0))
   )
-  (wire (pts (xy 54.61 121.92) (xy 71.12 121.92))
+  (wire (pts (xy 69.85 121.92) (xy 71.12 121.92))
     (stroke (width 0) (type default) (color 0 0 0 0))
   )
@@
     (stroke (width 0) (type default) (color 0 0 0 0))
   )
-  (wire (pts (xy 54.61 121.92) (xy 54.61 120.65))
+  (wire (pts (xy 69.85 121.92) (xy 69.85 120.65))
     (stroke (width 0) (type default) (color 0 0 0 0))
   )
@@
     (pin "1")
     (pin "2")
+  )
+  (symbol (lib_id "power:+3.3VA") (at 69.85 120.65 0) (unit 1)
+    (in_bom yes) (on_board yes)
+    (property "Reference" "#PWR?" (id 0) (at 69.85 124.46 0)
+      (effects (font (size 1.27 1.27)) hide)
+    )
+    (property "Value" "+3.3VA" (id 1) (at 64.77 119.38 0))
+    (property "Footprint" "" (id 2) (at 69.85 120.65 0)
+      (effects (font (size 1.27 1.27)) hide)
+    )
+    (property "Datasheet" "" (id 3) (at 69.85 120.65 0)
+      (effects (font (size 1.27 1.27)) hide)
+    )
+    (pin "1")
   )
   (symbol (lib_id "Connector:Conn_01x06_Female") (at 223.52 85.09 0) (unit 1)
@@
       (effects (font (size 1.27 1.27)) hide)
     )
-    (pin "1")
-  )
-  (symbol (lib_id "power:+3V3") (at 54.61 120.65 0) (unit 1)
-    (in_bom yes) (on_board yes) (fields_autoplaced)
-    (property "Reference" "#PWR09" (id 0) (at 54.61 124.46 0)
-      (effects (font (size 1.27 1.27)) hide)
-    )
-    (property "Value" "+3V3" (id 1) (at 54.61 115.57 0))
-    (property "Footprint" "" (id 2) (at 54.61 120.65 0)
-      (effects (font (size 1.27 1.27)) hide)
-    )
-    (property "Datasheet" "" (id 3) (at 54.61 120.65 0)
-      (effects (font (size 1.27 1.27)) hide)
-    )

Commit message: just ordered from JLCPCB
Other:
- note added: "Dual I2C Connections"
- note added: "Linear Regulator"
- note added: "Power demands on the ESP32 can be handled by its own linear regulator. This one is added to handle all breakouts, including the ADE7953, in hopes that the draw of the microcontroller is isolated from these."
- note added: "The I2C bus connection is used by the ADE7953, but here are 2 more that add more extensibility to the board as a whole. Once of these will likely be used by the PN532 Card Reader."
- company: (none) -> Corey Rice & MakeHaven
- title: (none) -> Breakout Connections & Power
- moved on the sheet: I2C-2, I2C-3, R7, R8, SPI-1, U3
