File: hardware/mh-custom-v2/esp32core.kicad_sch (KiCad schematic)
At the start: 1 part, among them U1 ESP32-DEVKITC-32D

Commit message: just ordered from JLCPCB
Other:
- company: (none) -> Corey Rice & MakeHaven
- title: (none) -> Connections to ESP32 Board
- moved on the sheet: U1
