File: hardware/mh-custom-v2/lightsounds.kicad_sch (KiCad schematic)
At the start: 26 parts, among them J1 Conn_01x03_Male, J2 Conn_01x03_Female, SW1 SW_DIP_x04, T1 AO3400A, T2 AO3400A, T5 AO3400A, T6 AO3400A

Commit message: b-silkscreen fixed
Other:
- note added: "Can read E-Stops seperately with the base config. Swapping two jumpers changes these to shared E-Stop readings and ability to reset ADE7953 in software."
- note added: "Leads to ADE7953 for second bypass jumper."
- note removed: "Can read E-Stops seperately with the base config. Swapping two jumpers changes these to shared E-Stop readings and ability to reset ADE7953."
Changed lines of the file:
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@@
     (stroke (width 0) (type default) (color 0 0 0 0))
   )
-  (wire (pts (xy 67.31 173.99) (xy 72.39 173.99))
+  (wire (pts (xy 59.69 173.99) (xy 72.39 173.99))
     (stroke (width 0) (type default) (color 0 0 0 0))
   )
@@
     (effects (font (size 2 2) (thickness 0.4) bold) (justify left bottom))
   )
+  (text "Leads to ADE7953 for second bypass jumper." (at 33.02 177.8 0)
+    (effects (font (size 1.27 1.27)) (justify left bottom))
+  )
   (text "4-DIP Switches" (at 44.45 49.53 0)
     (effects (font (size 2 2) (thickness 0.4) bold) (justify left bottom))
   )
-  (text "When reading LOW\nE-Stop is active." (at 50.8 180.34 0)
-    (effects (font (size 1.27 1.27)) (justify left bottom))
-  )
   (text "A single panel mounted Red/Green LED will indicate states\nof the system for every card read. These LEDs are cheap \nand relatively easy to find in pre-made panel mount packages."
     (at 196.85 96.52 0)
     (effects (font (size 1.27 1.27)) (justify left bottom))
   )
-  (text "Can read E-Stops \nseperately with \nthe base config. \n\nSwapping two jumpers \nchanges these to shared \nE-Stop readings and \nability to reset ADE7953."
+  (text "Can read E-Stops \nseperately with \nthe base config. \n\nSwapping two jumpers \nchanges these to shared \nE-Stop readings and \nability to reset ADE7953\nin software."
     (at 102.87 160.02 0)
     (effects (font (size 1.27 1.27)) (justify left bottom))
@@
     )
   )
-  (global_label "read-aux-E-Stop" (shape output) (at 67.31 173.99 180) (fields_autoplaced)
+  (global_label "read-aux-E-Stop" (shape output) (at 59.69 173.99 180) (fields_autoplaced)
     (effects (font (size 1.27 1.27)) (justify right))
-    (property "Intersheet References" "${INTERSHEET_REFS}" (id 0) (at 47.2983 173.9106 0)
+    (property "Intersheet References" "${INTERSHEET_REFS}" (id 0) (at 39.6783 173.9106 0)
       (effects (font (size 1.27 1.27)) (justify right) hide)
     )
@@
       (effects (font (size 1.27 1.27)) (justify left) hide)
     )
+  )
+  (symbol (lib_id "power:+3V3") (at 72.39 165.1 0) (unit 1)
+    (in_bom yes) (on_board yes) (fields_autoplaced)
+    (property "Reference" "#PWR04" (id 0) (at 72.39 168.91 0)
+      (effects (font (size 1.27 1.27)) hide)
+    )
+    (property "Value" "+3V3" (id 1) (at 72.39 160.02 0))
+    (property "Footprint" "" (id 2) (at 72.39 165.1 0)
+      (effects (font (size 1.27 1.27)) hide)
+    )
+    (property "Datasheet" "" (id 3) (at 72.39 165.1 0)
+      (effects (font (size 1.27 1.27)) hide)
+    )
+    (pin "1")
   )
   (symbol (lib_id "Device:R_US") (at 217.17 57.15 180) (unit 1)
@@
     (pin "1")
   )
-  (symbol (lib_id "power:+3V3") (at 217.17 52.07 0) (unit 1)
-    (in_bom yes) (on_board yes) (fields_autoplaced)
-    (property "Reference" "#PWR04" (id 0) (at 217.17 55.88 0)
-      (effects (font (size 1.27 1.27)) hide)
-    )
-    (property "Value" "+3V3" (id 1) (at 217.17 46.99 0))
-    (property "Footprint" "" (id 2) (at 217.17 52.07 0)
-      (effects (font (size 1.27 1.27)) hide)
-    )
-    (property "Datasheet" "" (id 3) (at 217.17 52.07 0)
-      (effects (font (size 1.27 1.27)) hide)
-    )
-    (pin "1")
-  )
   (symbol (lib_id "Device:LED_Dual_AKA") (at 250.19 109.22 180) (unit 1)
     (in_bom no) (on_board no) (fields_autoplaced)
@@
     (pin "1")
   )
+  (symbol (lib_id "power:+3V3") (at 217.17 52.07 0) (unit 1)
+    (in_bom yes) (on_board yes) (fields_autoplaced)
+    (property "Reference" "#PWR05" (id 0) (at 217.17 55.88 0)
+      (effects (font (size 1.27 1.27)) hide)
+    )
+    (property "Value" "+3V3" (id 1) (at 217.17 46.99 0))
+    (property "Footprint" "" (id 2) (at 217.17 52.07 0)
+      (effects (font (size 1.27 1.27)) hide)
+    )
+    (property "Datasheet" "" (id 3) (at 217.17 52.07 0)
+      (effects (font (size 1.27 1.27)) hide)
+    )
+    (pin "1")
+  )
   (symbol (lib_id "Device:Buzzer") (at 158.75 69.85 0) (unit 1)
     (in_bom yes) (on_board yes) (fields_autoplaced)
@@
       (effects (font (size 1.27 1.27)) hide)
     )
-    (pin "1")
-  )
-  (symbol (lib_id "power:+3V3") (at 72.39 165.1 0) (unit 1)
-    (in_bom yes) (on_board yes) (fields_autoplaced)
-    (property "Reference" "#PWR09" (id 0) (at 72.39 168.91 0)
-      (effects (font (size 1.27 1.27)) hide)
-    )
-    (property "Value" "+3V3" (id 1) (at 72.39 160.02 0))
-    (property "Footprint" "" (id 2) (at 72.39 165.1 0)
-      (effects (font (size 1.27 1.27)) hide)
-    )
-    (property "Datasheet" "" (id 3) (at 72.39 165.1 0)
-      (effects (font (size 1.27 1.27)) hide)
-    )

Commit message: applied workaround for 3.3v and 3v3 known bug: https://gitlab.com/kicad/libraries/kicad-symbols/-/issues/3153
Connections:
- net +3V3 renamed +3.3VA
Changed lines of the file:
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@@
     )
-  )
-  (symbol (lib_id "power:+3V3") (at 72.39 165.1 0) (unit 1)
-    (in_bom yes) (on_board yes) (fields_autoplaced)
-    (property "Reference" "#PWR04" (id 0) (at 72.39 168.91 0)
-      (effects (font (size 1.27 1.27)) hide)
-    )
-    (property "Value" "+3V3" (id 1) (at 72.39 160.02 0))
-    (property "Footprint" "" (id 2) (at 72.39 165.1 0)
-      (effects (font (size 1.27 1.27)) hide)
-    )
-    (property "Datasheet" "" (id 3) (at 72.39 165.1 0)
-      (effects (font (size 1.27 1.27)) hide)
-    )
-    (pin "1")
   )
   (symbol (lib_id "Device:R_US") (at 217.17 57.15 180) (unit 1)
@@
     (pin "3")
   )
-  (symbol (lib_id "power:+3V3") (at 72.39 121.92 0) (unit 1)
-    (in_bom yes) (on_board yes) (fields_autoplaced)
-    (property "Reference" "#PWR03" (id 0) (at 72.39 125.73 0)
-      (effects (font (size 1.27 1.27)) hide)
-    )
-    (property "Value" "+3V3" (id 1) (at 72.39 116.84 0))
-    (property "Footprint" "" (id 2) (at 72.39 121.92 0)
-      (effects (font (size 1.27 1.27)) hide)
-    )
-    (property "Datasheet" "" (id 3) (at 72.39 121.92 0)
-      (effects (font (size 1.27 1.27)) hide)
-    )
-    (pin "1")
-  )
   (symbol (lib_id "power:GND") (at 207.01 152.4 0) (unit 1)
     (in_bom yes) (on_board yes) (fields_autoplaced)
@@
     )
     (property "Datasheet" "" (id 3) (at 207.01 152.4 0)
-      (effects (font (size 1.27 1.27)) hide)
-    )
-    (pin "1")
-  )
-  (symbol (lib_id "power:+3V3") (at 217.17 52.07 0) (unit 1)
-    (in_bom yes) (on_board yes) (fields_autoplaced)
-    (property "Reference" "#PWR05" (id 0) (at 217.17 55.88 0)
-      (effects (font (size 1.27 1.27)) hide)
-    )
-    (property "Value" "+3V3" (id 1) (at 217.17 46.99 0))
-    (property "Footprint" "" (id 2) (at 217.17 52.07 0)
-      (effects (font (size 1.27 1.27)) hide)
-    )
-    (property "Datasheet" "" (id 3) (at 217.17 52.07 0)
       (effects (font (size 1.27 1.27)) hide)
     )
@@
     (pin "1")
   )
+  (symbol (lib_id "power:+3.3VA") (at 72.39 165.1 0) (unit 1)
+    (in_bom yes) (on_board yes)
+    (property "Reference" "#PWR?" (id 0) (at 72.39 168.91 0)
+      (effects (font (size 1.27 1.27)) hide)
+    )
+    (property "Value" "+3.3VA" (id 1) (at 67.31 163.83 0))
+    (property "Footprint" "" (id 2) (at 72.39 165.1 0)
+      (effects (font (size 1.27 1.27)) hide)
+    )
+    (property "Datasheet" "" (id 3) (at 72.39 165.1 0)
+      (effects (font (size 1.27 1.27)) hide)
+    )
+    (pin "1")
+  )
   (symbol (lib_id "power:+5V") (at 237.49 52.07 0) (unit 1)
     (in_bom yes) (on_board yes) (fields_autoplaced)
@@
     (pin "1")
   )
+  (symbol (lib_id "power:+3.3VA") (at 217.17 52.07 0) (unit 1)
+    (in_bom yes) (on_board yes)
+    (property "Reference" "#PWR?" (id 0) (at 217.17 55.88 0)
+      (effects (font (size 1.27 1.27)) hide)
+    )
+    (property "Value" "+3.3VA" (id 1) (at 212.09 50.8 0))
+    (property "Footprint" "" (id 2) (at 217.17 52.07 0)
+      (effects (font (size 1.27 1.27)) hide)
+    )
+    (property "Datasheet" "" (id 3) (at 217.17 52.07 0)
+      (effects (font (size 1.27 1.27)) hide)
+    )
+    (pin "1")
+  )
   (symbol (lib_id "power:GND") (at 50.8 77.47 0) (unit 1)
     (in_bom yes) (on_board yes)
@@
     (pin "3")
   )
+  (symbol (lib_id "power:+3.3VA") (at 72.39 121.92 0) (unit 1)
+    (in_bom yes) (on_board yes)
+    (property "Reference" "#PWR?" (id 0) (at 72.39 125.73 0)
+      (effects (font (size 1.27 1.27)) hide)
+    )
+    (property "Value" "+3.3VA" (id 1) (at 67.31 120.65 0))
+    (property "Footprint" "" (id 2) (at 72.39 121.92 0)
+      (effects (font (size 1.27 1.27)) hide)
+    )
+    (property "Datasheet" "" (id 3) (at 72.39 121.92 0)
+      (effects (font (size 1.27 1.27)) hide)
+    )
+    (pin "1")
+  )
   (symbol (lib_id "Connector:Conn_01x03_Female") (at 110.49 130.81 0) (unit 1)

Commit message: just ordered from JLCPCB
Other:
- company: (none) -> Corey Rice & MakeHaven
- title: (none) -> Onboard Lights, Sounds and Logic Level Converters
- moved on the sheet: BZ1, Boot-1, C1, C2, D1, E-Stop-1, E-Stop-2, EN-1, J1, J2, JP14, R1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
