File: hardware/mh-custom-v2/microcontroller.kicad_sch (KiCad schematic)
At the start: 0 parts

Commit message: just ordered from JLCPCB
Other:
- company: (none) -> Corey Rice & MakeHaven
Changed lines of the file:
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@@
 (kicad_sch (version 20211123) (generator eeschema)
   (paper "A4")
+  (title_block
+    (date "2022-10-09")
+    (rev "2")
+    (company "Corey Rice & MakeHaven")
+  )
   (sheet (at 96.52 124.46) (size 16.51 12.7) (fields_autoplaced)
     (stroke (width 0.1524) (type solid) (color 0 0 0 0))
