File: hardware/mh-custom-v2/stage2relay.kicad_sch (KiCad schematic)
At the start: 5 parts, among them SW2 SW_Push

Commit message: approaching ordering from JLCPCB
Parts:
- F1: JLCPCB Part # (none) -> C206977
- F2: JLBPCB Part # (none) -> C206977
- R31: footprint relay_Omron-MY2-02:relay-Omron-MY2-02 -> MY2-02 AC110 Omron:relay-Omron-MY2-02
Connections:
- net Member-E-Stop-aux-1: no longer R31.9
- net N/L2: no longer R31.14
- net mains-fused-N/L2: now also R31.14
- new net Member-E-Stop-aux-2: R31.9
Changed lines of the file:
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@@
     )
   )
-  (global_label "Member-E-Stop-aux-1" (shape input) (at 196.85 107.95 0) (fields_autoplaced)
+  (global_label "Member-E-Stop-aux-2" (shape input) (at 196.85 107.95 0) (fields_autoplaced)
     (effects (font (size 1.27 1.27)) (justify left))
     (property "Intersheet References" "${INTERSHEET_REFS}" (id 0) (at 222.7279 107.8706 0)
@@
     (property "Intersheet References" "${INTERSHEET_REFS}" (id 0) (at 111.2098 102.7906 0)
       (effects (font (size 1.27 1.27)) (justify left) hide)
-    )
-  )
-  (global_label "N{slash}L2" (shape passive) (at 68.58 140.97 180) (fields_autoplaced)
-    (effects (font (size 1.27 1.27)) (justify right))
-    (property "Intersheet References" "${INTERSHEET_REFS}" (id 0) (at 61.2683 140.8906 0)
-      (effects (font (size 1.27 1.27)) (justify right) hide)
     )
   )
@@
     (property "Intersheet References" "${INTERSHEET_REFS}" (id 0) (at 228.8964 62.1506 0)
       (effects (font (size 1.27 1.27)) (justify left) hide)
+    )
+  )
+  (global_label "mains-fused-N{slash}L2" (shape passive) (at 68.58 140.97 180) (fields_autoplaced)
+    (effects (font (size 1.27 1.27)) (justify right))
+    (property "Intersheet References" "${INTERSHEET_REFS}" (id 0) (at 47.3588 141.0494 0)
+      (effects (font (size 1.27 1.27)) (justify right) hide)
     )
   )
@@
       (effects (font (size 1.27 1.27)) (justify left))
     )
-    (property "Footprint" "relay_Omron-MY2-02:relay-Omron-MY2-02" (id 2) (at 93.98 110.49 0)
+    (property "Footprint" "MY2-02 AC110 Omron:relay-Omron-MY2-02" (id 2) (at 93.98 110.49 0)
       (effects (font (size 1.27 1.27)) hide)
     )
@@
     )
     (property "Datasheet" "~" (id 3) (at 205.74 156.21 0)
+      (effects (font (size 1.27 1.27)) hide)
+    )
+    (property "JLBPCB Part #" "C206977" (id 4) (at 205.74 156.21 90)
       (effects (font (size 1.27 1.27)) hide)
     )
@@
       (effects (font (size 1.27 1.27)) hide)
     )
+    (property "JLCPCB Part #" "C206977" (id 4) (at 205.74 153.67 90)
+      (effects (font (size 1.27 1.27)) hide)
+    )

Commit message: finalizing details of ordering from JLCPCB
Parts:
- F1: footprint Fuse:Fuseholder_Littelfuse_100_series_5x20mm -> Fuse:Fuseholder_Cylinder-5x20mm_Stelvio-Kontek_PTF78_Horizontal_Open; JLCPCB Part # C206977 -> C717030
- F2: footprint Fuse:Fuseholder_Littelfuse_100_series_5x20mm -> Fuse:Fuseholder_Cylinder-5x20mm_Stelvio-Kontek_PTF78_Horizontal_Open; JLBPCB Part # C206977 -> C717030
Changed lines of the file:
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@@
     (property "Reference" "F2" (id 0) (at 205.74 161.29 90))
     (property "Value" "Fuse" (id 1) (at 205.74 158.75 90))
-    (property "Footprint" "Fuse:Fuseholder_Littelfuse_100_series_5x20mm" (id 2) (at 205.74 157.988 90)
+    (property "Footprint" "Fuse:Fuseholder_Cylinder-5x20mm_Stelvio-Kontek_PTF78_Horizontal_Open" (id 2) (at 205.74 157.988 90)
       (effects (font (size 1.27 1.27)) hide)
     )
@@
       (effects (font (size 1.27 1.27)) hide)
     )
-    (property "JLBPCB Part #" "C206977" (id 4) (at 205.74 156.21 90)
+    (property "JLBPCB Part #" "C717030" (id 4) (at 205.74 156.21 90)
       (effects (font (size 1.27 1.27)) hide)
     )
@@
     (property "Reference" "F1" (id 0) (at 205.74 148.59 90))
     (property "Value" "Fuse" (id 1) (at 205.74 151.13 90))
-    (property "Footprint" "Fuse:Fuseholder_Littelfuse_100_series_5x20mm" (id 2) (at 205.74 155.448 90)
+    (property "Footprint" "Fuse:Fuseholder_Cylinder-5x20mm_Stelvio-Kontek_PTF78_Horizontal_Open" (id 2) (at 205.74 155.448 90)
       (effects (font (size 1.27 1.27)) hide)
     )
@@
       (effects (font (size 1.27 1.27)) hide)
     )
-    (property "JLCPCB Part #" "C206977" (id 4) (at 205.74 153.67 90)
+    (property "JLCPCB Part #" "C717030" (id 4) (at 205.74 153.67 90)
       (effects (font (size 1.27 1.27)) hide)
     )

Commit message: just ordered from JLCPCB
Other:
- company: (none) -> Corey Rice & MakeHaven
- title: (none) -> Stage 2 | Core 'Active Self-Latching' relay
Changed lines of the file:
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@@
 (kicad_sch (version 20211123) (generator eeschema)
   (paper "A4")
+  (title_block
+    (title "Stage 2 | Core 'Active Self-Latching' relay")
+    (date "2022-10-09")
+    (rev "2")
+    (company "Corey Rice & MakeHaven")
+    (comment 1 "Once activated, relay holds itself open with power ")
+    (comment 2 "Can be interrupted by E-Stops or the S1/'reset' relay")
+    (comment 3 "Fuses added to power inputs, to protect board from improper wiring")
+    (comment 4 "E-Stop low voltage light & switch logic shown for reference")
+  )
   (junction (at 115.57 138.43) (diameter 0) (color 0 0 0 0)
   )
