File: hardware/mh-custom-v2/stage3contactor.kicad_sch (KiCad schematic)
At the start: 9 parts, among them J10 Screw_Terminal_01x02, J11 Screw_Terminal_01x02, J12 Screw_Terminal_01x02, J5 Screw_Terminal_01x02, J6 Screw_Terminal_01x02, J7 Screw_Terminal_01x02, J8 Screw_Terminal_01x02, J9 Screw_Terminal_01x02

Commit message: just ordered from JLCPCB
Parts:
- J10, J11, J12, J5, J6, J7, J8, J9: JLCPCB Part # C8404 -> C8269
Other:
- company: (none) -> Corey Rice & MakeHaven
- title: (none) -> Stage 3 | Contactor to power the Tool
Changed lines of the file:
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@@
 (kicad_sch (version 20211123) (generator eeschema)
   (paper "A4")
+  (title_block
+    (title "Stage 3 | Contactor to power the Tool")
+    (date "2022-10-09")
+    (rev "2")
+    (company "Corey Rice & MakeHaven")
+    (comment 1 "The contactor actually controls the tool, and is activated by the 'OUT' line on the board")
+    (comment 2 "A fuse is added to protect the baord from improper wiring")
+    (comment 3 "Screw-terminals shown here, to connect to mains-level devices")
+    (comment 4 "Jumer the EStp3 if there will not be any secondary EStop used")
+  )
   (wire (pts (xy 212.09 114.3) (xy 213.36 114.3))
     (stroke (width 0) (type default) (color 0 0 0 0))
@@
       (effects (font (size 1.27 1.27)) hide)
     )
-    (property "JLCPCB Part #" "C8404" (id 4) (at 207.01 104.14 0)
+    (property "JLCPCB Part #" "C8269" (id 4) (at 207.01 104.14 0)
       (effects (font (size 1.27 1.27)) hide)
     )
@@
       (effects (font (size 1.27 1.27)) hide)
     )
-    (property "JLCPCB Part #" "C8404" (id 4) (at 207.01 134.62 0)
+    (property "JLCPCB Part #" "C8269" (id 4) (at 207.01 134.62 0)
       (effects (font (size 1.27 1.27)) hide)
     )
@@
       (effects (font (size 1.27 1.27)) hide)
     )
-    (property "JLCPCB Part #" "C8404" (id 4) (at 207.01 139.7 0)
+    (property "JLCPCB Part #" "C8269" (id 4) (at 207.01 139.7 0)
       (effects (font (size 1.27 1.27)) hide)
     )
@@
       (effects (font (size 1.27 1.27)) hide)
     )
-    (property "JLCPCB Part #" "C8404" (id 4) (at 207.01 124.46 0)
+    (property "JLCPCB Part #" "C8269" (id 4) (at 207.01 124.46 0)
       (effects (font (size 1.27 1.27)) hide)
     )
@@
       (effects (font (size 1.27 1.27)) hide)
     )
-    (property "JLCPCB Part #" "C8404" (id 4) (at 207.01 114.3 0)
+    (property "JLCPCB Part #" "C8269" (id 4) (at 207.01 114.3 0)
       (effects (font (size 1.27 1.27)) hide)
     )
@@
       (effects (font (size 1.27 1.27)) hide)
     )
-    (property "JLCPCB Part #" "C8404" (id 4) (at 207.01 109.22 0)
+    (property "JLCPCB Part #" "C8269" (id 4) (at 207.01 109.22 0)
       (effects (font (size 1.27 1.27)) hide)
     )
@@
       (effects (font (size 1.27 1.27)) hide)
     )
-    (property "JLCPCB Part #" "C8404" (id 4) (at 207.01 119.38 0)
+    (property "JLCPCB Part #" "C8269" (id 4) (at 207.01 119.38 0)
       (effects (font (size 1.27 1.27)) hide)
     )
@@
       (effects (font (size 1.27 1.27)) hide)
     )
-    (property "JLCPCB Part #" "C8404" (id 4) (at 207.01 129.54 0)
-      (effects (font (size 1.27 1.27)) hide)
-    )
+    (property "JLCPCB Part #" "C8269" (id 4) (at 207.01 129.54 0)
+      (effects (font (size 1.27 1.27)) hide)
+    )
